Commit message: Kinova camera launch and urdf changes (gripper etc) Also a pick detected object script in kinovademo

File: kinova_description/urdf/kinova_common.xacro (robot description, xacro)
@@ -15,4 +15,5 @@
 <xacro:include filename="$(find kinova_description)/urdf/kinova_inertial.xacro" />
     <xacro:property name="J_PI" value="3.1415926535897931" />
+    <xacro:property name="MAX_FINGER_TURN" value="0.008880645630600082" />
     <xacro:macro name="kinova_armlink" params="link_name link_mesh ring_mesh:=ring_big use_ring_mesh:=false mesh_no">
         <link name="${link_name}">
@@ -45,5 +46,5 @@
     </xacro:macro>
   <xacro:macro name="kinova_armjoint" params="joint_name type parent child joint_axis_xyz joint_origin_xyz joint_origin_rpy joint_lower_limit joint_upper_limit fixed:=false">
-    <joint name="${joint_name}" type="${type}">
+      <joint name="${joint_name}" type="${type}">
         <parent link="${parent}"/>
         <child link="${child}"/>
@@ -52,5 +53,5 @@
         <origin xyz="${joint_origin_xyz}" rpy="${joint_origin_rpy}"/>
         <dynamics damping="0.0" friction="0.0"/>
-     </joint>
+      </joint>
    <xacro:unless value="${fixed}">
      <transmission name="${prefix}_joint_1_trans">
@@ -64,5 +65,5 @@
         </actuator>
      </transmission>
-	<transmission name="${prefix}_joint_2_trans">
+	  <transmission name="${prefix}_joint_2_trans">
         <type>transmission_interface/SimpleTransmission</type>
         <joint name="${prefix}_joint_2">
